File: NanoDD/NanoDD.kicad_pcb (KiCad board)
At the start: 2 copper layers, 53.7 x 10.2 mm, 32 parts, among them J1 Screw_Terminal_01x02, J2 Screw_Terminal_01x02, J3 Conn_01x06, Q1 AO3401A, Q2 AO3401A, SW1 SW_SPDT, U1 BMP280, U2 MSP430G2452IRSA16, U3 XC6206PxxxMR, U4 ZD24C128A-XGMB

Commit message: Oops forgot to sleep and did all the layout
Parts:
- added TP1: TestPoint, TestPoint:TestPoint_Pad_1.5x1.5mm, F.Cu at (181.6, 92.7)
- added TP2: TestPoint, TestPoint:TestPoint_Pad_1.5x1.5mm, F.Cu at (185.4, 92.7)
- C1: renamed from C4; moved to B.Cu
- C2: renamed from C3; moved to B.Cu
- C3: renamed from C5; moved to B.Cu
- D1: value LED -> RED
- J2: renamed from J3; footprint Connector_Molex:Molex_PicoBlade_53398-0671_1x06-1MP_P1.25mm_Vertical -> Connector_Molex:Molex_PicoBlade_53047-0610_1x06_P1.25mm_Vertical
- R10: renamed from R8; moved to B.Cu
- R11: renamed from R7; moved to B.Cu
- R12: renamed from R6; moved to B.Cu
- R4: renamed from R3; moved to B.Cu
- R5: renamed from R1; moved to B.Cu
- R6: renamed from R4; moved to B.Cu
- R7: renamed from R5; moved to B.Cu
- moved R10 40.1 mm to (159.6, 93.0), turned to -90 degrees
- moved R12 36.2 mm to (159.6, 97.0), turned to 90 degrees
- moved R11 35.3 mm to (159.6, 95.0), turned to 90 degrees
- moved C3 28.2 mm to (176.8, 99.1)
- moved U4 27.8 mm to (166.0, 95.4)
- moved C2 26.4 mm to (178.2, 94.0), turned to 90 degrees
- moved R6 21.6 mm to (180.3, 99.9), turned to 90 degrees
- moved R7 21.1 mm to (179.0, 99.9), turned to 90 degrees
- moved R5 20.5 mm to (191.2, 99.9), turned to 180 degrees
- moved D1 19.0 mm to (188.5, 97.7), turned to 0 degrees
- moved C1 18.5 mm to (185.9, 93.1), turned to 135 degrees
- moved R4 16.3 mm to (191.2, 97.7)
- moved U2 15.6 mm to (176.8, 97.0)
- moved C4 14.5 mm to (169.0, 95.3)
- moved C5 12.2 mm to (165.6, 92.8), turned to 0 degrees
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- renumbered BZ2 to BZ1, C2 to C4, C1 to C5, H2 to H1, H1 to H2, J2 to J3, Q2 to Q1, Q1 to Q2, R11 to R1, R10 to R2, R9 to R3, R12 to R8, R13 to R9, U2 to U1, U1 to U2, U4 to U3, U3 to U4
Connections:
- J2 pad 2: /TEST_WTCK -> /SDA
- J2 pad 3: /RST_TDIO -> /SCL
- J2 pad 4: /SCL -> /RST_TDIO
- J2 pad 5: /SDA -> /TEST_WTCK
- U1 pad 1: /LED -> /AUX
- U1 pad 11: /PYRO1 -> /BUZZER
- U1 pad 12: /PYRO0 -> /PYRO1
- U1 pad 2: /BUZZER -> /CONT1
- U1 pad 3: unconnected-(U2-TA0.1/A2/CA2/P1.2-Pad3) -> /LED
- U1 pad 4: /VBAT_SENSE -> /PYRO0
- U1 pad 6: /CONT1 -> /VBAT_SENSE
Routing:
- net /CONT1: track 0.00 -> 33.9 mm, vias 0 -> 2
- net GND: track 2.24 -> 34.2 mm, vias 2 -> 8
- net /PYRO1: track 0.00 -> 27.8 mm
- net /SDA: track 0.00 -> 20.6 mm
- net /SCL: track 0.00 -> 19.6 mm, vias 0 -> 2
- net /RST_TDIO: track 0.00 -> 13.0 mm, vias 0 -> 1
- net /CONT0: track 0.00 -> 11.7 mm
- net /VBAT_SENSE: track 0.00 -> 11.2 mm, vias 0 -> 2
- net /TEST_WTCK: track 0.00 -> 11.0 mm, vias 0 -> 1
- net /PYRO0: track 0.00 -> 10.7 mm
- net /EMATCH0: track 0.00 -> 6.30 mm
- net /EMATCH1: track 0.00 -> 6.29 mm
- net /BUZZER: track 0.00 -> 5.70 mm, vias 0 -> 1
- net Net-(Q2-G): track 0.00 -> 5.11 mm
- net Net-(Q1-G): track 0.00 -> 5.08 mm
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Other:
- board size 53.7 x 10.2 mm -> 47.4 x 10.2 mm
- board text added: "+"
- board text added: ">:3"
- board text added: "AUX"
- board text added: "DROGUE"
- board text added: "GND"
- board text added: "JLCJLCJLCJLC"
- board text added: "MAIN"
- board text added: "NanoDeploy Altimeter v1.0"
- board text added: "by bry"
