File: NanoDD/NanoDD.kicad_sch (KiCad schematic)
At the start: 32 parts, among them J1 Screw_Terminal_01x02, J2 Screw_Terminal_01x02, J3 Conn_01x06, Q1 AO3401A, Q2 AO3401A, SW1 SW_SPDT, U1 BMP280, U2 MSP430G2452IRSA16, U3 XC6206PxxxMR, U4 ZD24C128A-XGMB

Commit message: Oops forgot to sleep and did all the layout
Parts:
- added TP1, TP2: TestPoint, TestPoint:TestPoint_Pad_1.5x1.5mm, symbol Connector:TestPoint
- D1: value LED -> RED
- J2: renamed from J3; footprint Connector_Molex:Molex_PicoBlade_53398-0671_1x06-1MP_P1.25mm_Vertical -> Connector_Molex:Molex_PicoBlade_53047-0610_1x06_P1.25mm_Vertical
- renumbered BZ2 to BZ1, C4 to C1, C3 to C2, C5 to C3, C2 to C4, C1 to C5, H2 to H1, H1 to H2, J2 to J3, Q2 to Q1, Q1 to Q2, R11 to R1, R8 to R10, R7 to R11, R6 to R12, R10 to R2, R9 to R3, R3 to R4, R1 to R5, R4 to R6, R5 to R7, R12 to R8, R13 to R9, U2 to U1, U1 to U2, U4 to U3, U3 to U4
Connections:
- net BUZZER: now also U1.11 (P2.7/XOUT); no longer U1.2 (TA0.0/A1/CA1/P1.1)
- net CONT1: now also U1.2 (TA0.0/A1/CA1/P1.1); no longer U1.6 (TMS/TA0.0/SCLK/A5/CA5/P1.5)
- net GND: now also TP1.1
- net LED: now also U1.3 (TA0.1/A2/CA2/P1.2); no longer U1.1 (TA0CLK/ACLK/A0/CA0/P1.0)
- net PYRO0: now also U1.4 (ADC10CLK/CAOUT/VREF-/VeREF-/A3/CA3/P1.3); no longer U1.12 (P2.6/XIN/TA0.1)
- net PYRO1: now also U1.12 (P2.6/XIN/TA0.1); no longer U1.11 (P2.7/XOUT)
- net RST_TDIO: now also J2.4 (Pin_4); no longer J2.3 (Pin_3)
- net SCL: now also J2.3 (Pin_3); no longer J2.4 (Pin_4)
- net SDA: now also J2.2 (Pin_2); no longer J2.5 (Pin_5)
- net TEST_WTCK: now also J2.5 (Pin_5); no longer J2.2 (Pin_2)
- net VBAT_SENSE: now also U1.6 (TMS/TA0.0/SCLK/A5/CA5/P1.5); no longer U1.4 (ADC10CLK/CAOUT/VREF-/VeREF-/A3/CA3/P1.3)
- new net AUX: TP2.1, U1.1 (TA0CLK/ACLK/A0/CA0/P1.0)
- no-connect marks 0 -> 2
Other:
- moved on the sheet: C1, C2, C3, J1, J2, J3, Q1, Q2, R1, R10, R11, R12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
