File: hardware/NanoProgrammer/NanoProgrammer.kicad_pcb (KiCad board)
At the start: 2 copper layers, 29.5 x 14.2 mm, 20 parts, among them J1 USB_A, J3 Conn_01x05, J4 Conn_01x04, U1 DS2480B+, U2 HT42B534

Commit message: huge bunch of uncommitted stuff idk what this is
Parts:
- added C5: 0.1uF, Capacitor_SMD:C_0402_1005Metric, F.Cu at (119.6, 62.8)
- added D1: RED, LED_SMD:LED_0603_1608Metric, F.Cu at (127.3, 70.3)
- added R5: 330, Resistor_SMD:R_0402_1005Metric, F.Cu at (122.9, 70.3)
- U2: footprint Package_SO:SO-8_3.9x4.9mm_P1.27mm -> Package_SO:SSOP-10_3.9x4.9mm_P1.00mm
- moved D3 14.7 mm to (109.2, 68.1), turned to 90 degrees
- moved D2 8.54 mm to (109.2, 63.0), turned to 90 degrees
- moved C1 7.34 mm to (111.5, 70.1), turned to 0 degrees
- moved C2 6.58 mm to (122.9, 69.1), turned to 0 degrees
- moved R1 4.29 mm to (127.8, 64.4), turned to 90 degrees
- moved C4 3.99 mm to (126.5, 64.4)
- moved R4 3.64 mm to (117.3, 70.1), turned to 180 degrees
- moved TP1 2.74 mm to (119.1, 65.8)
- moved TP2 2.65 mm to (119.1, 67.8)
- moved U1 2.54 mm to (114.3, 66.5)
- moved TP4 2.30 mm to (129.5, 64.5)
- moved TP5 2.30 mm to (129.5, 66.8)
- moved U2 1.98 mm to (122.9, 65.3), turned to -90 degrees
- moved R2 1.82 mm to (127.8, 66.4)
- moved R3 1.24 mm to (115.1, 70.1)
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Connections:
- C3 pad 1: /D- -> /D-R
- C4 pad 1: /D+ -> /D+R
- U2 pad 1: GND -> /D+R
- U2 pad 2: /TX -> +5V
- U2 pad 3: +5V -> +3V3
- U2 pad 4: /RX -> /TX
- U2 pad 5: /D+R -> /LED
- U2 pad 8: unconnected-(U2-V33O-Pad8) -> /RX
Routing:
- net /LED_TX: track 1.52 -> 11.8 mm
- net /LED: track 0.00 -> 8.62 mm, vias 0 -> 2
- net /RX: track 8.11 -> 16.2 mm
- net /LED_RX: track 1.50 -> 9.34 mm
- net /D-R: track 2.26 -> 9.47 mm
- net +5V: track 0.00 -> 4.01 mm, vias 0 -> 2
- net +3V3: track 0.00 -> 3.94 mm
- net /LED_USB: track 0.00 -> 3.11 mm
- net /D+: track 7.11 -> 4.78 mm
- net /D+R: track 2.15 -> 3.60 mm
- net /TX: track 13.8 -> 15.2 mm
- net GND: track 7.41 -> 7.35 mm, vias 4 -> 5
